File: n40a8/n40a8.kicad_pcb (KiCad board)
At the start: 2 copper layers, 288.1 x 92.9 mm, 93 parts, among them J1 Conn_01x16, SW1 SW_Push, SW10 SW_Push, SW11 SW_Push, SW12 SW_Push, SW13 SW_Push, SW14 SW_Push, SW15 SW_Push, SW16 SW_Push, SW17 SW_Push, SW18 SW_Push, SW19 SW_Push, SW2 SW_Push, SW20 SW_Push, SW21 SW_Push, SW22 SW_Push, SW23 SW_Push, SW24 SW_Push, SW25 SW_Push, SW26 SW_Push, SW27 SW_Push, SW28 SW_Push, SW29 SW_Push, SW3 SW_Push, SW30 SW_Push, SW31 SW_Push, SW32 SW_Push, SW33 SW_Push, SW34 SW_Push, SW35 SW_Push, SW36 SW_Push, SW37 SW_Push, SW38 SW_Push, SW39 SW_Push, SW4 SW_Push, SW40 SW_Push, SW41 SW_Push, SW42 SW_Push, SW43 SW_RST, SW44 SW_PWR, SW5 SW_Push, SW6 SW_Push, SW7 SW_Push, SW8 SW_Push, SW9 SW_Push, U1 BLE-Micro-Pro-2, U2 TPS61221

Commit message: move Diode
Parts:
- SW38: footprint cscslib:CPG151101S11_2u_RS -> cscslib:CPG151101S11_2u
- SW39: footprint cscslib:CPG151101S11_1.25u -> cscslib:CPG151101S11_2.25u
- SW40: footprint cscslib:CPG151101S11_2.25u_RS -> cscslib:CPG151101S11_1.25u
- moved SW39 63.2 mm to (200.3, 111.7), turned to 8 degrees
- moved D39 60.4 mm to (208.7, 111.8), turned to 98 degrees
- moved D40 35.9 mm to (241.7, 107.1)
- moved SW40 33.3 mm to (233.3, 107.1)
- moved D41 32.0 mm to (271.5, 106.0), turned to 90 degrees
- moved SW41 29.9 mm to (263.1, 104.8), turned to 0 degrees
- moved D20 4.29 mm to (215.2, 72.4)
- moved D21 4.29 mm to (234.1, 69.7)
- moved D7 4.29 mm to (189.0, 56.8)
- moved D19 4.29 mm to (196.4, 75.0)
- moved D22 4.29 mm to (252.9, 67.1)
- moved D10 4.29 mm to (245.6, 48.9)
- moved D9 4.29 mm to (226.7, 51.5)
- moved D8 4.29 mm to (207.9, 54.2)
- moved D15 4.29 mm to (112.3, 69.5)
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
Commit message: wired
Parts:
- J1: moved to F.Cu
- moved U1 2.98 mm to (311.9, 53.0), turned to 180 degrees
- moved D6 2.15 mm to (165.5, 59.0)
- moved D18 1.68 mm to (167.6, 78.5)
- moved D5 1.68 mm to (146.6, 56.3)
- moved D29 1.68 mm to (174.3, 98.7)
- moved D17 1.68 mm to (148.7, 75.8)
- moved D4 1.68 mm to (127.8, 53.7)
- moved D28 1.68 mm to (155.5, 96.0)
- moved D38 1.68 mm to (162.3, 116.2)
- moved D16 1.68 mm to (129.8, 73.2)
- moved D3 1.68 mm to (108.9, 51.0)
- moved D27 1.68 mm to (136.6, 93.4)
- moved D15 1.68 mm to (111.0, 70.5)
- moved D26 1.68 mm to (117.8, 90.7)
- moved D37 1.68 mm to (131.6, 111.9)
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Connections:
- SW37 pad 1: C2 -> C3
- SW38 pad 1: C3 -> C4
Routing:
- net R3: track 0.00 -> 258.5 mm
- net R1: track 0.00 -> 235.3 mm
- net R2: track 0.00 -> 228.7 mm
- net R0: track 0.00 -> 202.8 mm
- net C9: track 0.00 -> 100.7 mm, vias 0 -> 4
- net C8: track 0.00 -> 89.9 mm, vias 0 -> 4
- net C1: track 0.00 -> 84.8 mm, vias 0 -> 4
- net C10: track 0.00 -> 81.6 mm, vias 0 -> 4
- net C7: track 0.00 -> 77.9 mm, vias 0 -> 4
- net C4: track 0.00 -> 76.9 mm, vias 0 -> 4
- net C6: track 0.00 -> 73.9 mm, vias 0 -> 4
- net C3: track 0.00 -> 73.9 mm, vias 0 -> 4
- net C0: track 0.00 -> 72.6 mm, vias 0 -> 4
- net BAT: track 4.85 -> 69.2 mm
- net Net-(BT1-+): track 0.00 -> 51.7 mm
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Other:
- rule pad_to_mask_clearance: 0.051 -> 0.038
- rule solder_mask_min_width: 0.25 -> 0.1

Commit message: wiring complete
Parts:
- removed J1: Conn_01x16, cscslib:PinHeader_1x16_P1.27mm_Conthrough
- U1: moved to F.Cu
- moved SW44 189.1 mm to (144.7, 26.2), turned to 0 degrees
- moved SW43 183.2 mm to (156.0, 26.2), turned to 180 degrees
- moved L1 182.2 mm to (141.5, 34.0), turned to 90 degrees
- moved C2 177.9 mm to (146.0, 36.4), turned to 0 degrees
- moved U2 176.5 mm to (146.0, 34.0), turned to 180 degrees
- moved C1 175.1 mm to (146.0, 31.6), turned to 180 degrees
- moved BT1 163.5 mm to (150.5, 37.6), turned to 172 degrees
- moved U1 128.1 mm to (184.9, 36.5), turned to -82 degrees
Connections:
- U1 pad 10: C2 -> R2
- U1 pad 11: C1 -> R1
- U1 pad 12: C0 -> R0
- U1 pad 14: R3 -> C0
- U1 pad 15: R2 -> C1
- U1 pad 16: R1 -> C2
- U1 pad 17: R0 -> C3
- U1 pad 18: C10 -> C4
- U1 pad 19: C9 -> C5
- U1 pad 20: C8 -> C6
- U1 pad 5: C7 -> C10
- U1 pad 6: C6 -> C9
- U1 pad 7: C5 -> C8
- U1 pad 8: C4 -> C7
- U1 pad 9: C3 -> R3
Routing:
- net C0: track 72.6 -> 210.4 mm
- net C1: track 84.8 -> 201.4 mm
- net C2: track 51.4 -> 149.4 mm
- net R3: track 258.5 -> 342.1 mm, vias 0 -> 1
- net C3: track 73.9 -> 155.2 mm
- net C4: track 76.9 -> 141.4 mm
- net C10: track 81.6 -> 145.9 mm
- net R2: track 228.7 -> 290.7 mm, vias 0 -> 1
- net C5: track 51.4 -> 100.0 mm
- net C9: track 100.7 -> 145.7 mm
- net Net-(BT1-+): track 51.7 -> 13.0 mm
- net R1: track 235.3 -> 273.1 mm, vias 0 -> 1
- net RST: track 0.00 -> 37.2 mm
- net C6: track 73.9 -> 106.4 mm
- net C8: track 89.9 -> 118.5 mm
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Other:
- board size 288.1 x 92.9 mm -> 267.9 x 103.7 mm
- board text removed: "10"
- board text removed: "11"
- board text removed: "12"
- board text removed: "14"
- board text removed: "15"
- board text removed: "16"
- board text removed: "17"
- board text removed: "18"
- board text removed: "19"
- board text removed: "20"
- board text removed: "5"
- board text removed: "6"
- board text removed: "7"
- board text removed: "8"
- board text removed: "9"
- board text removed: "C0"
- board text removed: "C1"
- board text removed: "C2"
- board text removed: "C3"
- board text removed: "C4"
- board text removed: "C5"
- board text removed: "C6"
- board text removed: "C7"
- board text removed: "C8"
- board text removed: "C9"
- board text removed: "CA"
- board text removed: "GND"
- board text removed: "R0"
- board text removed: "R1"
- board text removed: "R2"
- board text removed: "R3"

Commit message: revise wiring
Parts:
- moved U1 1.31 mm to (184.7, 35.2)
Routing:
- net C6: track 106.4 -> 113.5 mm
- net RST: track 37.2 -> 39.9 mm
- net R2: track 290.7 -> 292.7 mm
- net C5: track 100.0 -> 101.9 mm
- net C7: track 92.1 -> 94.0 mm
- net C4: track 141.4 -> 143.0 mm
- net R3: track 342.1 -> 343.5 mm
- net C2: track 149.4 -> 150.7 mm
- net C3: track 155.2 -> 156.5 mm
- net C0: track 210.4 -> 211.7 mm
- net R1: track 273.1 -> 274.4 mm
- net C1: track 201.4 -> 202.6 mm
- net C8: track 118.5 -> 119.6 mm
- net C9: track 145.7 -> 146.3 mm
- net BAT: track 60.8 -> 60.2 mm
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Other:
- board text added: "JLCJLCJLCJLC"

Commit message: revise footprint
Parts:
- moved L1 1.93 mm to (139.6, 34.0)
- moved U2 1.93 mm to (144.1, 34.0)
- moved C1 1.93 mm to (144.1, 31.6)
- moved C2 1.93 mm to (144.1, 36.4)
Routing:
- net BAT: track 60.2 -> 62.3 mm
- net cell: track 14.6 -> 13.8 mm

Commit message: revise footprint for PCBA
Parts:
- SW1, SW10, SW11, SW12, SW13, SW14, SW15, SW16, SW17, SW18, SW19, SW2, SW20, SW21, SW22, SW23, SW24, SW25, SW26, SW27, SW28, SW29, SW3, SW30, SW31, SW32, SW33, SW34, SW35, SW36, SW37, SW38, SW39, SW4, SW40, SW41, SW42, SW5, SW6, SW7, SW8, SW9: moved to B.Cu
- turned SW1 to 180 degrees
- turned SW10 to -172 degrees
- turned SW11 to 180 degrees
- turned SW12 to 180 degrees
- turned SW13 to 180 degrees
- turned SW14 to 180 degrees
- turned SW15 to 172 degrees
- turned SW16 to 172 degrees
- turned SW17 to 172 degrees
- turned SW18 to 172 degrees
- turned SW19 to -172 degrees
- turned SW2 to 180 degrees
- turned SW20 to -172 degrees
- turned SW21 to -172 degrees
- turned SW22 to -172 degrees
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