File: n40a8/n40a8.kicad_pcb (KiCad board)
At the start: 2 copper layers, 267.9 x 103.7 mm, 92 parts, among them SW1 SW_Push, SW10 SW_Push, SW11 SW_Push, SW12 SW_Push, SW13 SW_Push, SW14 SW_Push, SW15 SW_Push, SW16 SW_Push, SW17 SW_Push, SW18 SW_Push, SW19 SW_Push, SW2 SW_Push, SW20 SW_Push, SW21 SW_Push, SW22 SW_Push, SW23 SW_Push, SW24 SW_Push, SW25 SW_Push, SW26 SW_Push, SW27 SW_Push, SW28 SW_Push, SW29 SW_Push, SW3 SW_Push, SW30 SW_Push, SW31 SW_Push, SW32 SW_Push, SW33 SW_Push, SW34 SW_Push, SW35 SW_Push, SW36 SW_Push, SW37 SW_Push, SW38 SW_Push, SW39 SW_Push, SW4 SW_Push, SW40 SW_Push, SW41 SW_Push, SW42 SW_Push, SW43 SW_RST, SW44 SW_PWR, SW5 SW_Push, SW6 SW_Push, SW7 SW_Push, SW8 SW_Push, SW9 SW_Push, U1 BLE-Micro-Pro-2, U2 TPS61221

Commit message: revise foot print for PCBA
Parts:
- C1, C2: value 10uF -> GRM188R60J106KE47D
- D1, D10, D11, D12, D13, D14, D15, D16, D17, D18, D19, D2, D20, D21, D22, D23, D24, D25, D26, D27, D28, D29, D3, D30, D31, D32, D33, D34, D35, D36, D37, D38, D39, D4, D40, D41, D42, D5, D6, D7, D8, D9: value D -> 1N4148W
- L1: value 4.7uH -> LQH3NPZ4R7MMEL
- SW1, SW10, SW11, SW12, SW13, SW14, SW15, SW16, SW17, SW18, SW19, SW2, SW20, SW21, SW22, SW23, SW24, SW25, SW26, SW27, SW28, SW29, SW3, SW30, SW31, SW32, SW33, SW34, SW35, SW36, SW37, SW38, SW39, SW4, SW40, SW41, SW42, SW5, SW6, SW7, SW8, SW9: value SW_Push -> CPG151101S11-16
- turned SW1 to 0 degrees
- turned SW10 to 8 degrees
- turned SW11 to 0 degrees
- turned SW12 to 0 degrees
- turned SW13 to 0 degrees
- turned SW14 to 0 degrees
- turned SW15 to -8 degrees
- turned SW16 to -8 degrees
- turned SW17 to -8 degrees
- turned SW18 to -8 degrees
- turned SW19 to 8 degrees
- turned SW2 to 0 degrees
- turned SW20 to 8 degrees
- turned SW21 to 8 degrees
- turned SW22 to 8 degrees
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
Commit message: revice for PCBA
Parts:
- added HOLE_M2: VAL**, cscslib:HOLE_M2, F.Cu at (275.0, 120.3)
- added HOLE_M2: VAL**, cscslib:HOLE_M2, F.Cu at (270.3, 33.3)
- added HOLE_M2: VAL**, cscslib:HOLE_M2, F.Cu at (64.3, 120.3)
- added HOLE_M2: VAL**, cscslib:HOLE_M2, F.Cu at (69.1, 33.3)
- moved BT1 11.0 mm to (161.5, 37.4)
- moved C2 7.23 mm to (151.2, 37.5)
- moved C1 7.23 mm to (151.2, 32.7)
- moved L1 7.23 mm to (146.8, 35.1)
- moved U2 7.23 mm to (151.2, 35.1)
- moved SW44 7.14 mm to (151.8, 26.2)
- moved SW43 6.55 mm to (162.5, 26.2)
- moved D3 1.19 mm to (108.9, 52.2)
- moved SW11 1.19 mm to (258.4, 47.6)
- moved D26 1.19 mm to (117.8, 91.9)
- moved D38 1.19 mm to (162.3, 117.4)
- moved D42 1.19 mm to (294.1, 108.3)
- moved SW16 1.19 mm to (123.1, 71.0)
- moved SW20 1.19 mm to (206.8, 73.6)
- moved D39 1.19 mm to (207.7, 114.3)
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Connections:
- U1 pad 20: C6 -> C10
- U1 pad 5: C10 -> C9
- U1 pad 6: C9 -> C8
- U1 pad 7: C8 -> C7
- U1 pad 8: C7 -> C6
Routing:
- net C6: track 113.5 -> 91.7 mm
- net C10: track 146.4 -> 163.0 mm
- net BAT: track 62.3 -> 55.3 mm
- net RST: track 39.9 -> 33.5 mm
- net Net-(BT1-+): track 13.0 -> 16.5 mm
- net C7: track 94.0 -> 91.1 mm
- net C8: track 119.6 -> 117.5 mm
- net C9: track 146.3 -> 144.8 mm
- net GND: track 1.92 -> 3.42 mm
- net C1: track 202.6 -> 203.9 mm
- net C0: track 211.7 -> 213.0 mm
- net cell: track 13.8 -> 15.0 mm
- net C4: track 143.0 -> 143.7 mm
- net R3: track 343.5 -> 344.1 mm
Other:
- board size 267.9 x 103.7 mm -> 267.9 x 104.9 mm
