File: n40a8/n40a8.kicad_pcb (KiCad board)
At the start: 2 copper layers, 267.9 x 104.9 mm, 96 parts, among them SW1 CPG151101S11-16, SW10 CPG151101S11-16, SW11 CPG151101S11-16, SW12 CPG151101S11-16, SW13 CPG151101S11-16, SW14 CPG151101S11-16, SW15 CPG151101S11-16, SW16 CPG151101S11-16, SW17 CPG151101S11-16, SW18 CPG151101S11-16, SW19 CPG151101S11-16, SW2 CPG151101S11-16, SW20 CPG151101S11-16, SW21 CPG151101S11-16, SW22 CPG151101S11-16, SW23 CPG151101S11-16, SW24 CPG151101S11-16, SW25 CPG151101S11-16, SW26 CPG151101S11-16, SW27 CPG151101S11-16, SW28 CPG151101S11-16, SW29 CPG151101S11-16, SW3 CPG151101S11-16, SW30 CPG151101S11-16, SW31 CPG151101S11-16, SW32 CPG151101S11-16, SW33 CPG151101S11-16, SW34 CPG151101S11-16, SW35 CPG151101S11-16, SW36 CPG151101S11-16, SW37 CPG151101S11-16, SW38 CPG151101S11-16, SW39 CPG151101S11-16, SW4 CPG151101S11-16, SW40 CPG151101S11-16, SW41 CPG151101S11-16, SW42 CPG151101S11-16, SW43 SW_RST, SW44 SW_PWR, SW5 CPG151101S11-16, SW6 CPG151101S11-16, SW7 CPG151101S11-16, SW8 CPG151101S11-16, SW9 CPG151101S11-16, U1 BLE-Micro-Pro-2, U2 TPS61221

Commit message: modified wiring
Parts:
- removed HOLE_M2 (x4): VAL**, cscslib:HOLE_M2
- added J1: Conn_01x01_Socket, cscslib:HOLE_M2, F.Cu at (69.1, 33.3)
- added J2: Conn_01x01_Socket, cscslib:HOLE_M2, F.Cu at (270.3, 33.3)
- added J3: Conn_01x01_Socket, cscslib:HOLE_M2, F.Cu at (64.3, 120.3)
- added J4: Conn_01x01_Socket, cscslib:HOLE_M2, F.Cu at (275.0, 120.3)
Connections:
- U1 pad 14: C0 -> C5
- U1 pad 15: C1 -> C4
- U1 pad 16: C2 -> C3
- U1 pad 17: C3 -> C2
- U1 pad 18: C4 -> C1
- U1 pad 19: C5 -> C0
Routing:
- net C0: track 213.0 -> 233.7 mm
- net C1: track 203.9 -> 221.5 mm
- net C2: track 151.0 -> 164.3 mm
- net C3: track 156.9 -> 165.0 mm
- net C8: track 117.5 -> 124.1 mm
- net C7: track 91.1 -> 97.4 mm
- net C4: track 143.7 -> 148.0 mm
- net C10: track 163.0 -> 166.6 mm
- net C5: track 101.7 -> 98.3 mm
- net RST: track 33.5 -> 30.1 mm
- net C9: track 144.8 -> 147.6 mm
- net C6: track 91.7 -> 94.2 mm
- net GND: track 3.42 -> 4.11 mm

Commit message: modified wiring
Parts:
- moved J2 0.60 mm to (270.3, 33.9)
- moved J1 0.60 mm to (69.1, 33.9)
- moved J4 0.60 mm to (275.0, 119.7)
- moved J3 0.60 mm to (64.3, 119.7)
Routing:
- net BAT: track 55.3 -> 77.3 mm
- net GND: track 4.11 -> 5.95 mm
- net R3: track 344.1 -> 345.1 mm
Other:
- outline, holes or cut-outs redrawn
