File: n40a8c/n40a8.kicad_pcb (KiCad board)
At the start: 2 copper layers, 267.9 x 104.9 mm, 107 parts, among them J1 Conn_01x01_Socket, J2 Conn_01x01_Socket, J3 Conn_01x01_Socket, J4 Conn_01x01_Socket, SW1 SW_Push, SW10 SW_Push, SW11 SW_Push, SW12 SW_Push, SW13 SW_Push, SW14 SW_Push, SW15 SW_Push, SW16 SW_Push, SW17 SW_Push, SW18 SW_Push, SW19 SW_Push, SW2 SW_Push, SW20 SW_Push, SW21 SW_Push, SW22 SW_Push, SW23 SW_Push, SW24 SW_Push, SW25 SW_Push, SW26 SW_Push, SW27 SW_Push, SW28 SW_Push, SW29 SW_Push, SW3 SW_Push, SW30 SW_Push, SW31 SW_Push, SW32 SW_Push, SW33 SW_Push, SW34 SW_Push, SW35 SW_Push, SW36 SW_Push, SW37 SW_Push, SW38 SW_Push, SW39 SW_Push, SW4 SW_Push, SW40 SW_Push, SW41 SW_Push, SW42 SW_Push, SW43 SW_PWR, SW5 SW_Push, SW6 SW_Push, SW7 SW_Push, SW8 SW_Push, SW9 SW_Push, U1 XIAO-nRF52840-SMD

Commit message: modify
Parts:
- moved DI2 142.1 mm to (171.5, 61.7), turned to -82 degrees
- moved DI4 134.8 mm to (178.8, 79.9), turned to -82 degrees
- moved DI8 130.6 mm to (183.5, 117.7), turned to -82 degrees
- moved DI6 123.2 mm to (190.9, 97.4), turned to -82 degrees
- moved DI7 47.1 mm to (42.9, 108.3)
- moved BT1 40.0 mm to (162.5, -2.59)
- moved DI5 37.2 mm to (42.3, 89.3)
- moved DI3 32.4 mm to (47.6, 69.7)
- moved DI1 27.2 mm to (47.6, 50.0)
Connections:
- U1 pad 1: ID 0 -> INTR
- U1 pad 2: ID 1 -> IO 1
- U1 pad 3: ID 2 -> IO 2
- U1 pad 4: ID 3 -> IO 3
- U1 pad 5: ID 5 -> IO 4
- U1 pad 6: ID 6 -> IO 5
- U1 pad 7: ID 7 -> IO 6
- U1 pad 8: INTR -> IO 7
- U1 pad 9: unconnected-(U1-P1.13_D8_SCK-Pad9) -> IO 0
Routing:
- net INTR: track 0.00 -> 271.9 mm, vias 0 -> 1
- net IO 1: track 118.9 -> 327.9 mm, vias 6 -> 8
- net IO 2: track 159.3 -> 343.6 mm, vias 6 -> 8
- net IO 3: track 137.7 -> 319.9 mm, vias 7 -> 9
- net IO 6: track 109.8 -> 277.5 mm, vias 6 -> 8
- net IO 5: track 169.9 -> 333.7 mm, vias 7 -> 9
- net IO 4: track 56.0 -> 134.7 mm, vias 3 -> 5
- net IO 0: track 79.1 -> 99.4 mm, vias 4 -> 5
- net IO 7: track 56.0 -> 74.8 mm, vias 3 -> 4
- net Net-(D13-K): track 136.7 -> 121.7 mm
- net Net-(D30-K): track 116.1 -> 101.3 mm
- net Net-(D1-K): track 129.9 -> 119.7 mm
- net Net-(D35-K): track 128.8 -> 119.8 mm
- net Net-(D39-K): track 118.9 -> 111.2 mm
- net Net-(D18-A): track 0.00 -> 6.24 mm
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
Commit message: revise wiring
Parts:
- SW43: footprint cscslib:TACT_SWITCH_TVBP06 -> cscslib:SLIDE_SWITCH_SK-12D01
- U1: moved to F.Cu
- moved DS3 148.5 mm to (172.3, 80.4)
- moved DS1 143.4 mm to (169.5, 56.2)
- moved DS5 139.5 mm to (160.0, 98.4)
- moved DS7 120.9 mm to (138.7, 111.0)
- moved DS2 58.3 mm to (248.8, 50.0)
- moved DS4 48.3 mm to (259.0, 69.7)
- moved DS6 34.0 mm to (275.0, 89.3)
- moved DS8 9.54 mm to (298.8, 108.3)
- moved SW43 5.98 mm to (156.6, 26.8), turned to 0 degrees
- turned U1 to 0 degrees
Connections:
- SW1 pad 1: IO 2 -> IO 7
- SW13 pad 1: IO 2 -> IO 7
- SW14 pad 1: IO 3 -> IO 6
- SW15 pad 1: IO 4 -> IO 5
- SW16 pad 1: IO 5 -> IO 4
- SW17 pad 1: IO 6 -> IO 3
- SW18 pad 1: IO 7 -> IO 2
- SW2 pad 1: IO 3 -> IO 6
- SW24 pad 1: IO 1 -> IO 7
- SW25 pad 1: IO 3 -> IO 6
- SW26 pad 1: IO 4 -> IO 5
- SW27 pad 1: IO 5 -> IO 4
- SW28 pad 1: IO 6 -> IO 3
- SW29 pad 1: IO 7 -> IO 1
- SW3 pad 1: IO 4 -> IO 5
- SW35 pad 1: IO 1 -> IO 7
- SW36 pad 1: IO 2 -> IO 6
- SW37 pad 1: IO 5 -> IO 4
- SW38 pad 1: IO 6 -> IO 1
- SW4 pad 1: IO 5 -> IO 4
- SW5 pad 1: IO 6 -> IO 3
- SW6 pad 1: IO 7 -> IO 2
Routing:
- net IO 7: track 74.8 -> 417.3 mm, vias 4 -> 6
- net IO 2: track 343.6 -> 162.9 mm, vias 8 -> 6
- net IO 1: track 327.9 -> 197.6 mm, vias 8 -> 7
- net INTR: track 271.9 -> 154.8 mm, vias 1 -> 0
- net IO 4: track 134.7 -> 244.2 mm, vias 5 -> 6
- net IO 6: track 277.5 -> 346.3 mm, vias 8 -> 7
- net IO 3: track 319.9 -> 255.1 mm, vias 9 -> 8
- net IO 0: track 99.4 -> 80.2 mm
- net Net-(D14-A): track 6.24 -> 0.00 mm
- net Net-(D39-K): track 111.2 -> 116.4 mm
- net IO 5: track 333.7 -> 336.4 mm, vias 9 -> 8
- net Net-(D1-K): track 119.7 -> 118.4 mm
- net Net-(D13-K): track 121.7 -> 120.6 mm
- net Net-(D30-K): track 101.3 -> 101.8 mm

Commit message: use SMD
Parts:
- U1: footprint cscslib:XIAO-nRF52840-SMD -> cscslib:XIAO-nRF52840-DIP
- moved DI2 122.0 mm to (292.9, 50.0), turned to -90 degrees
- moved DI4 115.1 mm to (293.5, 69.7), turned to -90 degrees
- moved DI8 114.5 mm to (297.7, 108.3), turned to -90 degrees
- moved DI6 104.7 mm to (295.3, 89.3), turned to -90 degrees
- moved DS8 7.14 mm to (298.8, 101.2)
- moved DS1 4.50 mm to (168.5, 60.6), turned to -98 degrees
- moved DS7 3.13 mm to (138.7, 114.1), turned to -98 degrees
- moved DS3 1.80 mm to (170.5, 80.1), turned to -98 degrees
- moved DS5 1.71 mm to (158.4, 97.6), turned to -98 degrees
- moved U1 1.57 mm to (177.4, 34.5)
Connections:
- U1 pad 2: IO 1 -> IO 7
- U1 pad 3: IO 2 -> IO 6
- U1 pad 4: IO 3 -> IO 5
- U1 pad 6: IO 5 -> IO 3
- U1 pad 7: IO 6 -> IO 2
- U1 pad 8: IO 7 -> IO 1
Routing:
- net INTR: track 154.8 -> 428.1 mm, vias 0 -> 1
- net IO 0: track 80.2 -> 144.8 mm
- net IO 1: track 197.6 -> 251.6 mm
- net IO 6: track 346.3 -> 386.6 mm, vias 7 -> 8
- net IO 2: track 162.9 -> 200.0 mm, vias 6 -> 7
- net IO 3: track 255.1 -> 290.2 mm, vias 8 -> 9
- net Net-(D39-K): track 116.4 -> 98.3 mm
- net Net-(D10-K): track 119.0 -> 105.9 mm
- net Net-(D30-K): track 101.8 -> 88.7 mm
- net IO 4: track 244.2 -> 253.7 mm, vias 6 -> 5
- net Net-(D19-K): track 106.2 -> 98.5 mm
- net Net-(D14-A): track 0.00 -> 6.24 mm
- net IO 5: track 336.4 -> 342.4 mm
- net Net-(D1-K): track 118.4 -> 121.3 mm
- net Net-(D13-K): track 120.6 -> 123.4 mm
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- added copper zone on B.Cu, net GND
- added copper zone on F.Cu, net GND
Other:
- outline, holes or cut-outs redrawn

Commit message: rewire
Parts:
- removed BT1: Battery_Cell, Battery:BatteryHolder_Keystone_2466_1xAAA
- removed SW43: SW_PWR, cscslib:SLIDE_SWITCH_SK-12D01
- moved U1 3.57 mm to (173.8, 34.5)
Routing:
- net IO 1: track 251.6 -> 264.5 mm
- net IO 0: track 144.8 -> 154.7 mm
- net IO 2: track 200.0 -> 204.4 mm
- net IO 7: track 419.4 -> 422.9 mm
- net IO 6: track 386.6 -> 389.5 mm
- net INTR: track 428.1 -> 430.6 mm
- net IO 3: track 290.2 -> 292.7 mm
- net IO 5: track 342.4 -> 344.8 mm
- net IO 4: track 253.7 -> 255.7 mm
Other:
- outline, holes or cut-outs redrawn
