File: n40a8c/n40a8.kicad_sch (KiCad schematic)
At the start: 107 parts, among them J1 Conn_01x01_Socket, J2 Conn_01x01_Socket, J3 Conn_01x01_Socket, J4 Conn_01x01_Socket, SW1 SW_Push, SW10 SW_Push, SW11 SW_Push, SW12 SW_Push, SW13 SW_Push, SW14 SW_Push, SW15 SW_Push, SW16 SW_Push, SW17 SW_Push, SW18 SW_Push, SW19 SW_Push, SW2 SW_Push, SW20 SW_Push, SW21 SW_Push, SW22 SW_Push, SW23 SW_Push, SW24 SW_Push, SW25 SW_Push, SW26 SW_Push, SW27 SW_Push, SW28 SW_Push, SW29 SW_Push, SW3 SW_Push, SW30 SW_Push, SW31 SW_Push, SW32 SW_Push, SW33 SW_Push, SW34 SW_Push, SW35 SW_Push, SW36 SW_Push, SW37 SW_Push, SW38 SW_Push, SW39 SW_Push, SW4 SW_Push, SW40 SW_Push, SW41 SW_Push, SW42 SW_Push, SW43 SW_PWR, SW5 SW_Push, SW6 SW_Push, SW7 SW_Push, SW8 SW_Push, SW9 SW_Push, U1 XIAO-nRF52840-SMD

Commit message: modify
Parts:
- renumbered D6 to D1, D18 to D13, D17 to D14, D16 to D15, D15 to D16, D14 to D17, D13 to D18, D5 to D2, D29 to D24, D28 to D25, D27 to D26, D26 to D27, D25 to D28, D24 to D29, D4 to D3, D38 to D35, D37 to D36, D36 to D37, D35 to D38, D3 to D4, D2 to D5, D1 to D6, SW6 to SW1, SW18 to SW13, SW17 to SW14, SW16 to SW15, SW15 to SW16, SW14 to SW17, SW13 to SW18, SW5 to SW2, SW29 to SW24, SW28 to SW25, SW27 to SW26, SW26 to SW27, SW25 to SW28, SW24 to SW29, SW4 to SW3, SW38 to SW35, SW37 to SW36, SW36 to SW37, SW35 to SW38, SW3 to SW4, SW2 to SW5, SW1 to SW6
Connections:
- net ID 0 is gone; now on net INTR: U1.1 (P0.02_A0_D0)
- net ID 1 is gone; now on net IO 1: U1.2 (P0.03_A1_D1)
- net ID 2 is gone; now on net IO 2: U1.3 (P0.28_A2_D2)
- net ID 3 is gone; now on net IO 3: U1.4 (P0.29_A3_D3)
- net ID 5 is gone; now on net IO 4: U1.5 (P0.04_A4_D4_SDA)
- net ID 6 is gone; now on net IO 5: U1.6 (P0.05_A5_D5_SCL)
- net ID 7 is gone; now on net IO 6: U1.7 (P1.11_D6_TX)
- net INTR: no longer U1.8 (P1.12_D7_RX)
- net IO 0: now also U1.9 (P1.13_D8_SCK)
- net IO 2: no longer SW37.1
- net IO 4: now also SW37.1
- net IO 5: no longer SW36.1
- net IO 6: now also SW36.1; no longer SW35.1
- net IO 7: now also SW35.1, U1.8 (P1.12_D7_RX)
- no-connect marks 9 -> 8
Other:
- moved on the sheet: D1, D13, D14, D15, D16, D17, D18, D2, D24, D25, D26, D27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

Commit message: use SMD
Parts:
- SW1, SW12: footprint cscslib:CPG151101S11_1u -> cscslib:CPG151101S11_1.5u
- SW13, SW34: footprint cscslib:CPG151101S11_1u -> cscslib:CPG151101S11_1.75u
- SW23, SW24, SW39: footprint cscslib:CPG151101S11_1u -> cscslib:CPG151101S11_2.25u
- SW35, SW36, SW37, SW40, SW41, SW42: footprint cscslib:CPG151101S11_1u -> cscslib:CPG151101S11_1.25u
- SW38: footprint cscslib:CPG151101S11_1u -> cscslib:CPG151101S11_2u
- U1: footprint cscslib:XIAO-nRF52840-SMD -> cscslib:XIAO-nRF52840-DIP
Connections:
- net IO 1: now also U1.8 (P1.12_D7_RX); no longer U1.2 (P0.03_A1_D1)
- net IO 2: now also U1.7 (P1.11_D6_TX); no longer U1.3 (P0.28_A2_D2)
- net IO 3: now also U1.6 (P0.05_A5_D5_SCL); no longer U1.4 (P0.29_A3_D3)
- net IO 5: now also U1.4 (P0.29_A3_D3); no longer U1.6 (P0.05_A5_D5_SCL)
- net IO 6: now also U1.3 (P0.28_A2_D2); no longer U1.7 (P1.11_D6_TX)
- net IO 7: now also U1.2 (P0.03_A1_D1); no longer U1.8 (P1.12_D7_RX)
Changed lines of the file:
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@@
 	(global_label "IO 3"
 		(shape bidirectional)
-		(at 21.59 44.45 180)
+		(at 21.59 52.07 180)
 		(fields_autoplaced yes)
 		(effects
@@
 		)
 		(property "Intersheetrefs" "${INTERSHEET_REFS}"
-			(at 14.1941 44.45 0)
+			(at 14.1941 52.07 0)
 			(effects
 				(font
@@
 	(global_label "IO 2"
 		(shape bidirectional)
-		(at 21.59 40.64 180)
+		(at 21.59 55.88 180)
 		(fields_autoplaced yes)
 		(effects
@@
 		)
 		(property "Intersheetrefs" "${INTERSHEET_REFS}"
-			(at 14.1941 40.64 0)
+			(at 14.1941 55.88 0)
 			(effects
 				(font
@@
 	(global_label "IO 5"
 		(shape bidirectional)
-		(at 21.59 52.07 180)
+		(at 21.59 44.45 180)
 		(fields_autoplaced yes)
 		(effects
@@
 		)
 		(property "Intersheetrefs" "${INTERSHEET_REFS}"
-			(at 14.1941 52.07 0)
+			(at 14.1941 44.45 0)
 			(effects
 				(font
@@
 	(global_label "IO 6"
 		(shape bidirectional)
-		(at 21.59 55.88 180)
+		(at 21.59 40.64 180)
 		(fields_autoplaced yes)
 		(effects
@@
 		)
 		(property "Intersheetrefs" "${INTERSHEET_REFS}"
-			(at 14.1941 55.88 0)
+			(at 14.1941 40.64 0)
 			(effects
 				(font
@@
 	(global_label "IO 7"
 		(shape bidirectional)
-		(at 68.58 55.88 0)
+		(at 21.59 36.83 180)
 		(fields_autoplaced yes)
 		(effects
@@
 				(size 1.27 1.27)
 			)
-			(justify left)
+			(justify right)
 		)
 		(property "Intersheetrefs" "${INTERSHEET_REFS}"
-			(at 75.9759 55.88 0)
+			(at 14.1941 36.83 0)
 			(effects
 				(font
 					(size 1.27 1.27)
 				)
-				(justify left)
+				(justify right)
 				(hide yes)
 			)
@@
 	(global_label "IO 1"
 		(shape bidirectional)
-		(at 21.59 36.83 180)
+		(at 68.58 55.88 0)
 		(fields_autoplaced yes)
 		(effects
@@
 				(size 1.27 1.27)
 			)
-			(justify right)
+			(justify left)
 		)
 		(property "Intersheetrefs" "${INTERSHEET_REFS}"
-			(at 14.1941 36.83 0)
+			(at 75.9759 55.88 0)
 			(effects
 				(font
 					(size 1.27 1.27)
 				)
-				(justify right)
+				(justify left)
 				(hide yes)
 			)
@@
 			)
 		)
-		(property "Footprint" "cscslib:CPG151101S11_1u"
+		(property "Footprint" "cscslib:CPG151101S11_1.5u"
 			(at 309.88 99.06 0)
 			(effects
@@
 			)
 		)
-		(property "Footprint" "cscslib:CPG151101S11_1u"
+		(property "Footprint" "cscslib:CPG151101S11_1.25u"
 			(at 289.56 160.02 0)
 			(effects
@@
 			)
 		)
-		(property "Footprint" "cscslib:CPG151101S11_1u"
+		(property "Footprint" "cscslib:CPG151101S11_2.25u"
 			(at 198.12 160.02 0)
 			(effects
@@
 			)
 		)
-		(property "Footprint" "cscslib:CPG151101S11_1u"
+		(property "Footprint" "cscslib:CPG151101S11_1.75u"
 			(at 36.195 119.38 0)
 			(effects
@@
 			)
 		)
-		(property "Footprint" "cscslib:CPG151101S11_1u"
+		(property "Footprint" "cscslib:CPG151101S11_2.25u"
 			(at 309.88 119.38 0)
 			(effects
@@
 			)
 		)
-		(property "Footprint" "cscslib:CPG151101S11_1u"
+		(property "Footprint" "cscslib:CPG151101S11_1.25u"
 			(at 36.195 160.02 0)
 			(effects
@@
 			)
 		)
-		(property "Footprint" "cscslib:CPG151101S11_1u"
+		(property "Footprint" "cscslib:CPG151101S11_1.75u"
 			(at 289.56 139.7 0)
 			(effects
@@
 			)
 		)
-		(property "Footprint" "cscslib:CPG151101S11_1u"
+		(property "Footprint" "cscslib:CPG151101S11_1.25u"
 			(at 97.155 160.02 0)
 			(effects
@@
 			)
 		)
-		(property "Footprint" "cscslib:CPG151101S11_1u"
+		(property "Footprint" "cscslib:CPG151101S11_1.5u"
 			(at 36.195 99.06 0)
 			(effects
@@
 			)
 		)
-		(property "Footprint" "cscslib:CPG151101S11_1u"
+		(property "Footprint" "cscslib:CPG151101S11_1.25u"
 			(at 259.08 160.02 0)
 			(effects
@@
 			)
 		)
-		(property "Footprint" "cscslib:CPG151101S11_1u"
+		(property "Footprint" "cscslib:CPG151101S11_2u"
 			(at 158.115 160.02 0)
 			(effects
@@
 			)
 		)
-		(property "Footprint" "cscslib:CPG151101S11_1u"
+		(property "Footprint" "cscslib:CPG151101S11_1.25u"
 			(at 56.515 160.02 0)
 			(effects
@@
 			)
 		)
-		(property "Footprint" "cscslib:XIAO-nRF52840-SMD"
+		(property "Footprint" "cscslib:XIAO-nRF52840-DIP"
 			(at 36.83 39.37 0)
 			(effects
@@
 			)
 		)
-		(property "Footprint" "cscslib:CPG151101S11_1u"
+		(property "Footprint" "cscslib:CPG151101S11_2.25u"
 			(at 36.195 139.7 0)
 			(effects
@@
 			)
 		)
-		(property "Footprint" "cscslib:CPG151101S11_1u"
+		(property "Footprint" "cscslib:CPG151101S11_1.25u"
 			(at 218.44 160.02 0)
 			(effects

Commit message: rewire
Parts:
- removed BT1: Battery_Cell, Battery:BatteryHolder_Keystone_2466_1xAAA, symbol Device:Battery_Cell
- added J5: Conn_01x02_Pin, symbol Connector:Conn_01x02_Pin
Connections:
- net GND: no longer U1.16 (GND)
- net VCC: now also U1.14 (5V); no longer U1.12 (3V3)
- net at SW43.2 (B): now also J5.1 (Pin_1)
- net RST: no longer names the net of U1.21 (RESET)
- net cell renamed BAT+
- new net 3V3: U1.12 (3V3)
- new net BAT-: J5.2 (Pin_2), U1.16 (GND)
Other:
- moved on the sheet: D1, D13, D14, D15, D16, D17, D18, D2, D24, D25, D26, D27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
