File: n40a8c/n40a8c.kicad_pcb (KiCad board)
At the start: 2 copper layers, 267.9 x 104.9 mm, 109 parts, among them J1 Conn_01x02_Pin, J2 Conn_01x02_Pin, J3 Conn_01x01_Socket, J4 Conn_01x01_Socket, J5 Conn_01x01_Socket, J6 Conn_01x01_Socket, SW1 SW_Push, SW10 SW_Push, SW11 SW_Push, SW12 SW_Push, SW13 SW_Push, SW14 SW_Push, SW15 SW_Push, SW16 SW_Push, SW17 SW_Push, SW18 SW_Push, SW19 SW_Push, SW2 SW_Push, SW20 SW_Push, SW21 SW_Push, SW22 SW_Push, SW23 SW_Push, SW24 SW_Push, SW25 SW_Push, SW26 SW_Push, SW27 SW_Push, SW28 SW_Push, SW29 SW_Push, SW3 SW_Push, SW30 SW_Push, SW31 SW_Push, SW32 SW_Push, SW33 SW_Push, SW34 SW_Push, SW35 SW_Push, SW36 SW_Push, SW37 SW_Push, SW38 SW_Push, SW39 SW_Push, SW4 SW_Push, SW40 SW_Push, SW41 SW_Push, SW42 SW_Push, SW43 SW_PWR, SW5 SW_Push, SW6 SW_Push, SW7 SW_Push, SW8 SW_Push, SW9 SW_Push, U1 XIAO-nRF52840-SMD

Commit message: change pin assign.
Connections:
- U1 pad 10: unconnected-(U1-P1.14_D9_MISO-Pad10) -> IO 1
- U1 pad 11: unconnected-(U1-P1.15_D10_MOSI-Pad11) -> IO 0
- U1 pad 7: IO 2 -> unconnected-(U1-P1.11_D6_TX-Pad7)_1
- U1 pad 8: IO 1 -> unconnected-(U1-P1.12_D7_RX-Pad8)
- U1 pad 9: IO 0 -> IO 2
Routing:
- net IO 2: track 220.6 -> 250.7 mm
- net IO 1: track 203.3 -> 213.4 mm
- net IO 0: track 129.1 -> 137.4 mm
- net GND: vias 0 -> 1
Other:
- board text added: "n40a8c Rev 1.0 Apr.2025 Designed ny @_hatano_"
- board text removed: "n40a8c Rev 1.0 2025/04/01 Designed ny @_hatano_"
