File: n40a8c/n40a8c.kicad_sch (KiCad schematic)
At the start: 109 parts, among them J1 Conn_01x02_Pin, J2 Conn_01x02_Pin, J3 Conn_01x01_Socket, J4 Conn_01x01_Socket, J5 Conn_01x01_Socket, J6 Conn_01x01_Socket, SW1 SW_Push, SW10 SW_Push, SW11 SW_Push, SW12 SW_Push, SW13 SW_Push, SW14 SW_Push, SW15 SW_Push, SW16 SW_Push, SW17 SW_Push, SW18 SW_Push, SW19 SW_Push, SW2 SW_Push, SW20 SW_Push, SW21 SW_Push, SW22 SW_Push, SW23 SW_Push, SW24 SW_Push, SW25 SW_Push, SW26 SW_Push, SW27 SW_Push, SW28 SW_Push, SW29 SW_Push, SW3 SW_Push, SW30 SW_Push, SW31 SW_Push, SW32 SW_Push, SW33 SW_Push, SW34 SW_Push, SW35 SW_Push, SW36 SW_Push, SW37 SW_Push, SW38 SW_Push, SW39 SW_Push, SW4 SW_Push, SW40 SW_Push, SW41 SW_Push, SW42 SW_Push, SW43 SW_PWR, SW5 SW_Push, SW6 SW_Push, SW7 SW_Push, SW8 SW_Push, SW9 SW_Push, U1 XIAO-nRF52840-SMD

Commit message: change pin assign.
Connections:
- net IO 0: now also U1.11 (P1.15_D10_MOSI); no longer U1.9 (P1.13_D8_SCK)
- net IO 1: now also U1.10 (P1.14_D9_MISO); no longer U1.8 (P1.12_D7_RX)
- net IO 2: now also U1.9 (P1.13_D8_SCK); no longer U1.7 (P1.11_D6_TX)
Changed lines of the file:
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@@
 	)
 	(no_connect
-		(at 68.58 48.26)
+		(at 68.58 55.88)
 	)
 	(no_connect
@@
 	)
 	(no_connect
-		(at 68.58 44.45)
+		(at 21.59 55.88)
 	)
 	(no_connect
@@
 	(global_label "IO 0"
 		(shape bidirectional)
+		(at 68.58 44.45 0)
+		(fields_autoplaced yes)
+		(effects
+			(font
+				(size 1.27 1.27)
+			)
+			(justify left)
+		)
+		(property "Intersheetrefs" "${INTERSHEET_REFS}"
+			(at 75.9759 44.45 0)
+			(effects
+				(font
+					(size 1.27 1.27)
+				)
+				(justify left)
+				(hide yes)
+			)
+		)
+	)
+	(global_label "IO 2"
+		(shape bidirectional)
 		(at 68.58 52.07 0)
 		(fields_autoplaced yes)
@@
 				)
 				(justify left)
-				(hide yes)
-			)
-		)
-	)
-	(global_label "IO 2"
-		(shape bidirectional)
-		(at 21.59 55.88 180)
-		(fields_autoplaced yes)
-		(effects
-			(font
-				(size 1.27 1.27)
-			)
-			(justify right)
-		)
-		(property "Intersheetrefs" "${INTERSHEET_REFS}"
-			(at 14.1941 55.88 0)
-			(effects
-				(font
-					(size 1.27 1.27)
-				)
-				(justify right)
 				(hide yes)
 			)
@@
 	(global_label "IO 1"
 		(shape bidirectional)
-		(at 68.58 55.88 0)
-		(fields_autoplaced yes)
-		(effects
-			(font
-				(size 1.27 1.27)
-			)
-			(justify left)
-		)
-		(property "Intersheetrefs" "${INTERSHEET_REFS}"
-			(at 75.9759 55.88 0)
-			(effects
-				(font
+		(at 68.58 48.26 0)
+		(fields_autoplaced yes)
+		(effects
+			(font
+				(size 1.27 1.27)
+			)
+			(justify left)
+		)
+		(property "Intersheetrefs" "${INTERSHEET_REFS}"
+			(at 75.9759 48.26 0)
+			(effects
+				(font
